File: arduino-shield.sch (KiCad schematic (older format))
At the start: 1 part

Commit message: misc
Connections:
- net at SHIELD1.GND1: now also SHIELD1.GND2, SHIELD1.SP6 (Gnd)
Changed lines of the file:
@@
 	1    0    0    -1
 $EndComp
+Wire Wire Line
+	4700 4100 4700 4200
+Wire Wire Line
+	6600 2900 6600 3000
+Wire Wire Line
+	6600 3000 4500 3000
+Wire Wire Line
+	4500 3000 4500 4100
+Wire Wire Line
+	4500 4100 4700 4100
 $EndSCHEMATC
