File: arduino-shield.kicad_pcb (KiCad board)
At the start: 2 copper layers, 410 parts

Commit message: 3nd commit
Parts:
- removed the 1 at (82.5, 88.9)
- removed the 211 at (82.5, 114.3)
- removed the 211 at (128.3, 109.2)
- removed 2110, 21100, 21101, 21102, 21103, 21104, 21105, 21106, 21107, 21108, 21109, 2111, 21110, 21111, 21112, 21113, 21114, 21115, 21116, 21117, 21118, 21119, 2112, 21120, 21121, 21122, 21123, 21124, 21125, 21126, 21127, 21128, 21129, 2113, 21130, 21131, 21132, 21133, 21134, 21135, 21136, 21137, 21138, 21139, 2114, 21140, 21141, 21142, 21143, 21144, 2115, 2116, 2117, 2118, 2119, 2120, 2121, 2122, 2123, 2124, 2125, 2126, 2127, 2128, 2129, 2130, 2131, 2132, 2133, 2134, 2135, 2136, 2137, 2138, 2139, 2140, 2141, 2142, 2143, 2144, 2145, 2146, 2147, 2148, 2149, 2150, 2151, 2152, 2153, 2154, 2155, 2156, 2157, 2158, 2159, 2160, 2161, 2162, 2163, 2164, 2165, 2166, 2167, 2168, 2169, 2170, 2171, 2172, 2173, 2174, 2175, 2176, 2177, 2178, 2179, 2180, 2181, 2182, 2183, 2184, 2185, 2186, 2187, 2188, 2189, 2190, 2191, 2192, 2193, 2194, 2195, 2196, 2197, 2198, 2199: , Connect:1pin
- removed the 212 at (85.1, 114.3)
- removed the 212 at (130.8, 109.2)
- removed the 213 at (87.6, 114.3)
- removed the 213 at (133.3, 109.2)
- removed the 214 at (90.2, 114.3)
- removed the 214 at (135.9, 109.2)
- removed the 215 at (92.7, 114.3)
- removed the 215 at (138.4, 109.2)
- removed the 217 at (97.8, 114.3)
- removed the 217 at (82.5, 111.8)
- removed the 218 at (100.3, 114.3)
- removed the 218 at (85.1, 111.8)
- removed the 219 at (102.9, 114.3)
- removed the 219 at (87.6, 111.8)
- removed the 3 at (87.6, 88.9)
- added 1: , Connect:1pin, F.Cu at (81.3, 88.9)
- added 1: , Connect:1pin, F.Cu at (81.3, 86.4)
- added 144: , Connect:1pin, F.Cu at (127.0, 101.6)
- added 168: , Connect:1pin, F.Cu at (124.5, 104.1)
- added 192: , Connect:1pin, F.Cu at (121.9, 106.7)
- added 211: , Connect:1pin, F.Cu at (106.7, 109.2)
- added 212: , Connect:1pin, F.Cu at (109.2, 109.2)
- added 213: , Connect:1pin, F.Cu at (111.8, 109.2)
- added 214: , Connect:1pin, F.Cu at (114.3, 109.2)
- added 215: , Connect:1pin, F.Cu at (116.8, 109.2)
- added 217: , Connect:1pin, F.Cu at (121.9, 109.2)
- added 218: , Connect:1pin, F.Cu at (124.5, 109.2)
- added 219: , Connect:1pin, F.Cu at (127.0, 109.2)
- added 241: , Connect:1pin, F.Cu at (119.4, 111.8)
- added 242: , Connect:1pin, F.Cu at (121.9, 111.8)
- added 243: , Connect:1pin, F.Cu at (124.5, 111.8)
- added 244: , Connect:1pin, F.Cu at (127.0, 111.8)
- added 245: , Connect:1pin, F.Cu at (129.5, 111.8)
- added 246: , Connect:1pin, F.Cu at (132.1, 111.8)
- added 247: , Connect:1pin, F.Cu at (134.6, 111.8)
- added 248: , Connect:1pin, F.Cu at (137.2, 111.8)
- added 249: , Connect:1pin, F.Cu at (139.7, 111.8)
- added 250: , Connect:1pin, F.Cu at (144.8, 121.9)
- added 250: , Connect:1pin, F.Cu at (144.8, 119.4)
- added 250: , Connect:1pin, F.Cu at (144.8, 116.8)
- added 250: , Connect:1pin, F.Cu at (144.8, 114.3)
- added 250: , Connect:1pin, F.Cu at (144.8, 111.8)
- added 250: , Connect:1pin, F.Cu at (142.2, 111.8)
- added 251: , Connect:1pin, F.Cu at (81.3, 114.3)
- added 252: , Connect:1pin, F.Cu at (83.8, 114.3)
- added 253: , Connect:1pin, F.Cu at (86.4, 114.3)
- added 254: , Connect:1pin, F.Cu at (88.9, 114.3)
- added 255: , Connect:1pin, F.Cu at (91.4, 114.3)
- added 256: , Connect:1pin, F.Cu at (94.0, 114.3)
- added 257: , Connect:1pin, F.Cu at (96.5, 114.3)
- added 258: , Connect:1pin, F.Cu at (99.1, 114.3)
- added 259: , Connect:1pin, F.Cu at (101.6, 114.3)
- added 260: , Connect:1pin, F.Cu at (104.1, 114.3)
- added 261: , Connect:1pin, F.Cu at (106.7, 114.3)
- added 262: , Connect:1pin, F.Cu at (109.2, 114.3)
- added 263: , Connect:1pin, F.Cu at (111.8, 114.3)
- added 264: , Connect:1pin, F.Cu at (114.3, 114.3)
- added 265: , Connect:1pin, F.Cu at (116.8, 114.3)
- added 266: , Connect:1pin, F.Cu at (119.4, 114.3)
- added 267: , Connect:1pin, F.Cu at (121.9, 114.3)
- added 268: , Connect:1pin, F.Cu at (124.5, 114.3)
- added 269: , Connect:1pin, F.Cu at (127.0, 114.3)
- added 270: , Connect:1pin, F.Cu at (129.5, 114.3)
- added 271: , Connect:1pin, F.Cu at (132.1, 114.3)
- added 272: , Connect:1pin, F.Cu at (134.6, 114.3)
- added 273: , Connect:1pin, F.Cu at (137.2, 114.3)
- added 274: , Connect:1pin, F.Cu at (139.7, 114.3)
- added 275: , Connect:1pin, F.Cu at (142.2, 114.3)
- added 276: , Connect:1pin, F.Cu at (81.3, 116.8)
- added 277: , Connect:1pin, F.Cu at (83.8, 116.8)
- added 278: , Connect:1pin, F.Cu at (86.4, 116.8)
- added 279: , Connect:1pin, F.Cu at (88.9, 116.8)
- added 280: , Connect:1pin, F.Cu at (91.4, 116.8)
- added 281: , Connect:1pin, F.Cu at (94.0, 116.8)
- added 282: , Connect:1pin, F.Cu at (96.5, 116.8)
- added 283: , Connect:1pin, F.Cu at (99.1, 116.8)
- added 284: , Connect:1pin, F.Cu at (101.6, 116.8)
- added 285: , Connect:1pin, F.Cu at (104.1, 116.8)
- added 286: , Connect:1pin, F.Cu at (106.7, 116.8)
- added 287: , Connect:1pin, F.Cu at (109.2, 116.8)
- added 288: , Connect:1pin, F.Cu at (111.8, 116.8)
- added 289: , Connect:1pin, F.Cu at (114.3, 116.8)
- added 290: , Connect:1pin, F.Cu at (116.8, 116.8)
- added 291: , Connect:1pin, F.Cu at (119.4, 116.8)
- added 292: , Connect:1pin, F.Cu at (121.9, 116.8)
- added 293: , Connect:1pin, F.Cu at (124.5, 116.8)
- added 294: , Connect:1pin, F.Cu at (127.0, 116.8)
- added 295: , Connect:1pin, F.Cu at (129.5, 116.8)
- added 296: , Connect:1pin, F.Cu at (132.1, 116.8)
- added 297: , Connect:1pin, F.Cu at (134.6, 116.8)
- added 298: , Connect:1pin, F.Cu at (137.2, 116.8)
- added 299: , Connect:1pin, F.Cu at (139.7, 116.8)
- added 3: , Connect:1pin, F.Cu at (81.3, 81.3)
- added 3: , Connect:1pin, F.Cu at (83.8, 81.3)
- added 3: , Connect:1pin, F.Cu at (86.4, 81.3)
- added 3: , Connect:1pin, F.Cu at (88.9, 81.3)
- added 3: , Connect:1pin, F.Cu at (81.3, 83.8)
- added 3: , Connect:1pin, F.Cu at (83.8, 83.8)
- added 3: , Connect:1pin, F.Cu at (86.4, 83.8)
- added 3: , Connect:1pin, F.Cu at (88.9, 83.8)
- added 3: , Connect:1pin, F.Cu at (86.4, 88.9)
- added 300: , Connect:1pin, F.Cu at (142.2, 116.8)
- added 301: , Connect:1pin, F.Cu at (81.3, 119.4)
- added 302: , Connect:1pin, F.Cu at (83.8, 119.4)
- added 303: , Connect:1pin, F.Cu at (86.4, 119.4)
- added 304: , Connect:1pin, F.Cu at (88.9, 119.4)
- added 305: , Connect:1pin, F.Cu at (91.4, 119.4)
- added 306: , Connect:1pin, F.Cu at (94.0, 119.4)
- added 307: , Connect:1pin, F.Cu at (96.5, 119.4)
- added 308: , Connect:1pin, F.Cu at (99.1, 119.4)
- added 309: , Connect:1pin, F.Cu at (101.6, 119.4)
- added 310: , Connect:1pin, F.Cu at (104.1, 119.4)
- added 311: , Connect:1pin, F.Cu at (106.7, 119.4)
- added 312: , Connect:1pin, F.Cu at (109.2, 119.4)
- added 313: , Connect:1pin, F.Cu at (111.8, 119.4)
- added 314: , Connect:1pin, F.Cu at (114.3, 119.4)
- added 315: , Connect:1pin, F.Cu at (116.8, 119.4)
- added 316: , Connect:1pin, F.Cu at (119.4, 119.4)
- added 317: , Connect:1pin, F.Cu at (121.9, 119.4)
- added 318: , Connect:1pin, F.Cu at (124.5, 119.4)
- added 319: , Connect:1pin, F.Cu at (127.0, 119.4)
- added 320: , Connect:1pin, F.Cu at (129.5, 119.4)
- added 321: , Connect:1pin, F.Cu at (132.1, 119.4)
- added 322: , Connect:1pin, F.Cu at (134.6, 119.4)
- added 323: , Connect:1pin, F.Cu at (137.2, 119.4)
- added 324: , Connect:1pin, F.Cu at (139.7, 119.4)
- added 325: , Connect:1pin, F.Cu at (142.2, 119.4)
- added 326: , Connect:1pin, F.Cu at (81.3, 121.9)
- added 327: , Connect:1pin, F.Cu at (83.8, 121.9)
- added 328: , Connect:1pin, F.Cu at (86.4, 121.9)
- added 329: , Connect:1pin, F.Cu at (88.9, 121.9)
- added 330: , Connect:1pin, F.Cu at (91.4, 121.9)
- added 331: , Connect:1pin, F.Cu at (94.0, 121.9)
- added 332: , Connect:1pin, F.Cu at (96.5, 121.9)
- added 333: , Connect:1pin, F.Cu at (99.1, 121.9)
- added 334: , Connect:1pin, F.Cu at (101.6, 121.9)
- added 335: , Connect:1pin, F.Cu at (104.1, 121.9)
- added 336: , Connect:1pin, F.Cu at (106.7, 121.9)
- added 337: , Connect:1pin, F.Cu at (109.2, 121.9)
- added 338: , Connect:1pin, F.Cu at (111.8, 121.9)
- added 339: , Connect:1pin, F.Cu at (114.3, 121.9)
- added 340: , Connect:1pin, F.Cu at (116.8, 121.9)
- added 341: , Connect:1pin, F.Cu at (119.4, 121.9)
- added 342: , Connect:1pin, F.Cu at (121.9, 121.9)
- added 343: , Connect:1pin, F.Cu at (124.5, 121.9)
- added 344: , Connect:1pin, F.Cu at (127.0, 121.9)
- added 345: , Connect:1pin, F.Cu at (129.5, 121.9)
- added 346: , Connect:1pin, F.Cu at (132.1, 121.9)
- added 347: , Connect:1pin, F.Cu at (134.6, 121.9)
- added 348: , Connect:1pin, F.Cu at (137.2, 121.9)
- added 349: , Connect:1pin, F.Cu at (139.7, 121.9)
- added 350: , Connect:1pin, F.Cu at (142.2, 121.9)
- added 351: , Connect:1pin, F.Cu at (81.3, 124.5)
- added 352: , Connect:1pin, F.Cu at (83.8, 124.5)
- added 353: , Connect:1pin, F.Cu at (86.4, 124.5)
- added 354: , Connect:1pin, F.Cu at (88.9, 124.5)
- added 355: , Connect:1pin, F.Cu at (91.4, 124.5)
- added 356: , Connect:1pin, F.Cu at (94.0, 124.5)
- added 357: , Connect:1pin, F.Cu at (96.5, 124.5)
- added 358: , Connect:1pin, F.Cu at (99.1, 124.5)
- added 359: , Connect:1pin, F.Cu at (101.6, 124.5)
- added 360: , Connect:1pin, F.Cu at (104.1, 124.5)
- added 361: , Connect:1pin, F.Cu at (106.7, 124.5)
- added 362: , Connect:1pin, F.Cu at (109.2, 124.5)
- added 363: , Connect:1pin, F.Cu at (111.8, 124.5)
- added 364: , Connect:1pin, F.Cu at (114.3, 124.5)
- added 365: , Connect:1pin, F.Cu at (116.8, 124.5)
- added 366: , Connect:1pin, F.Cu at (119.4, 124.5)
- added 367: , Connect:1pin, F.Cu at (121.9, 124.5)
- added 368: , Connect:1pin, F.Cu at (124.5, 124.5)
- added 369: , Connect:1pin, F.Cu at (127.0, 124.5)
- added 370: , Connect:1pin, F.Cu at (129.5, 124.5)
- added 371: , Connect:1pin, F.Cu at (132.1, 124.5)
- added 372: , Connect:1pin, F.Cu at (134.6, 124.5)
- added 373: , Connect:1pin, F.Cu at (137.2, 124.5)
- added 374: , Connect:1pin, F.Cu at (139.7, 124.5)
- added 375: , Connect:1pin, F.Cu at (142.2, 124.5)
- added 376: , Connect:1pin, F.Cu at (81.3, 127.0)
- added 377: , Connect:1pin, F.Cu at (83.8, 127.0)
- added 378: , Connect:1pin, F.Cu at (86.4, 127.0)
- added 379: , Connect:1pin, F.Cu at (88.9, 127.0)
- added 380: , Connect:1pin, F.Cu at (91.4, 127.0)
- added 381: , Connect:1pin, F.Cu at (94.0, 127.0)
- added 382: , Connect:1pin, F.Cu at (81.3, 129.5)
- added 382: , Connect:1pin, F.Cu at (83.8, 129.5)
- added 382: , Connect:1pin, F.Cu at (86.4, 129.5)
- added 382: , Connect:1pin, F.Cu at (88.9, 129.5)
- added 382: , Connect:1pin, F.Cu at (104.1, 129.5)
- added 382: , Connect:1pin, F.Cu at (101.6, 129.5)
- added 382: , Connect:1pin, F.Cu at (99.1, 129.5)
- added 382: , Connect:1pin, F.Cu at (96.5, 129.5)
- added 382: , Connect:1pin, F.Cu at (96.5, 127.0)
- added 383: , Connect:1pin, F.Cu at (99.1, 127.0)
- added 384: , Connect:1pin, F.Cu at (101.6, 127.0)
- added 385: , Connect:1pin, F.Cu at (104.1, 127.0)
- added 386: , Connect:1pin, F.Cu at (106.7, 127.0)
- added 387: , Connect:1pin, F.Cu at (109.2, 127.0)
- added 388: , Connect:1pin, F.Cu at (111.8, 127.0)
- added 389: , Connect:1pin, F.Cu at (114.3, 127.0)
- added 390: , Connect:1pin, F.Cu at (116.8, 127.0)
- added 391: , Connect:1pin, F.Cu at (119.4, 127.0)
- added 392: , Connect:1pin, F.Cu at (121.9, 127.0)
- added 393: , Connect:1pin, F.Cu at (124.5, 127.0)
- added 394: , Connect:1pin, F.Cu at (127.0, 127.0)
- added 395: , Connect:1pin, F.Cu at (129.5, 127.0)
- added 396: , Connect:1pin, F.Cu at (132.1, 127.0)
- added 397: , Connect:1pin, F.Cu at (134.6, 127.0)
- added 398: , Connect:1pin, F.Cu at (137.2, 127.0)
- added 399: , Connect:1pin, F.Cu at (139.7, 127.0)
- added 400: , Connect:1pin, F.Cu at (142.2, 127.0)
- moved 25 59.7 mm to (142.2, 88.9)
- moved 50 57.2 mm to (142.2, 91.4)
- moved 49 57.2 mm to (139.7, 91.4)
- moved 75 54.7 mm to (142.2, 94.0)
- moved 73 54.7 mm to (137.2, 94.0)
- moved 74 54.7 mm to (139.7, 94.0)
- moved 100 52.1 mm to (142.2, 96.5)
- moved 97 52.1 mm to (134.6, 96.5)
- moved 98 52.1 mm to (137.2, 96.5)
- moved 99 52.1 mm to (139.7, 96.5)
- moved 121 49.6 mm to (132.1, 99.1)
- moved 125 49.6 mm to (142.2, 99.1)
- moved 122 49.6 mm to (134.6, 99.1)
- moved 123 49.6 mm to (137.2, 99.1)
- moved 124 49.6 mm to (139.7, 99.1)
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
Commit message: misc
Parts:
- removed the 250 at (144.8, 121.9)
- removed the 250 at (144.8, 119.4)
- removed the 250 at (144.8, 116.8)
- removed the 250 at (144.8, 114.3)
- removed the 250 at (144.8, 111.8)
- removed 275, 300, 325, 350: , Connect:1pin
- removed the 3 at (81.3, 81.3)
- removed the 3 at (83.8, 81.3)
- removed the 3 at (86.4, 81.3)
- removed the 3 at (88.9, 81.3)
- removed the 3 at (81.3, 83.8)
- removed the 3 at (83.8, 83.8)
- removed the 3 at (86.4, 83.8)
- removed the 3 at (88.9, 83.8)
- removed the 382 at (81.3, 129.5)
- removed the 382 at (83.8, 129.5)
- removed the 382 at (86.4, 129.5)
- removed the 382 at (88.9, 129.5)
- removed the 382 at (101.6, 129.5)
- removed the 382 at (99.1, 129.5)
Connections:
- SHIELD1 pad GND2: Net-(SHIELD1-PadGND2) -> Net-(SHIELD1-PadGND1)
- SHIELD1 pad SP6: Net-(SHIELD1-PadSP6) -> Net-(SHIELD1-PadGND1)

Commit message: KiCad 6.0.3 format.
Other:
- net class Default removed
